File: KeychronQ9OrthoIntegrated.kicad_pcb (KiCad board)
At the start: 2 copper layers, 309.6 x 76.2 mm, 162 parts, among them J1 Conn_01x07, J3 Conn_01x05, U1 XC6206PxxxMR, U2 SRV05-4, U3 RP2040, U4 W25Q128JVS, Y1 Crystal_GND24

Commit message: add encoders, ground fill, production files
Parts:
- added SW1: RotaryEncoder_Switch, PCM_marbastlib-various:ROT_Alps_EC11E-Switch, F.Cu at (315.9, 25.4)
- added SW2: RotaryEncoder_Switch, PCM_marbastlib-various:ROT_Alps_EC11E-Switch, F.Cu at (315.9, 49.2)
- moved C11 9.94 mm to (322.1, 57.5), turned to 90 degrees
- moved U4 7.91 mm to (320.2, 63.2), turned to 90 degrees
- moved C8 4.80 mm to (313.6, 67.8), turned to -90 degrees
- moved C10 2.71 mm to (309.6, 75.1)
- moved C12 2.69 mm to (306.0, 75.3)
- moved Y1 2.69 mm to (308.0, 73.5)
- moved C15 2.53 mm to (307.4, 56.2)
- moved C16 2.53 mm to (308.4, 56.2)
- moved C4 2.02 mm to (305.6, 70.2)
- moved C13 2.01 mm to (306.6, 71.1)
- moved R9 2.01 mm to (305.6, 72.7)
- moved R3 1.93 mm to (321.4, 40.6)
- moved R6 1.93 mm to (323.3, 39.5)
- moved U3 1.82 mm to (307.5, 63.8)
- moved R4 1.79 mm to (323.3, 40.6)
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Connections:
- U3 pad 2: unconnected-(U3-GPIO0-Pad2) -> ENC1B
- U3 pad 3: unconnected-(U3-GPIO1-Pad3) -> ENC1A
- U3 pad 4: unconnected-(U3-GPIO2-Pad4) -> ENC2A
- U3 pad 5: Col 13 -> ENC2B
- U3 pad 6: Col 14 -> Col 13
- U3 pad 7: Col 15 -> Col 14
- U3 pad 8: Col 16 -> Col 15
- U3 pad 9: unconnected-(U3-GPIO7-Pad9) -> Col 16
Routing:
- net ENC1B: track 0.00 -> 42.2 mm, vias 0 -> 2
- net ENC1A: track 0.00 -> 39.3 mm, vias 0 -> 2
- net Row 2: track 316.3 -> 336.2 mm
- net Col 16: track 348.7 -> 367.1 mm
- net Row 1: track 340.6 -> 357.7 mm
- net ENC2B: track 0.00 -> 16.3 mm, vias 0 -> 1
- net GND: track 92.8 -> 108.4 mm, vias 22 -> 57
- net Q_CLK: track 7.92 -> 20.5 mm
- net Q_IO3: track 8.94 -> 21.5 mm
- net Q_SEL: track 42.8 -> 55.1 mm
- net Q_IO0: track 7.37 -> 19.5 mm
- net ENC2A: track 0.00 -> 10.9 mm, vias 0 -> 1
- net +3V3: track 155.1 -> 145.5 mm, vias 5 -> 3
- net +1V1: track 32.9 -> 26.5 mm
- net unconnected-(U3-GPIO8-Pad11): track 5.41 -> 0.00 mm
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