File: Q9-Chimera/Q9-Chimera.kicad_pcb (KiCad board)
At the start: 2 copper layers, 309.6 x 76.2 mm, 194 parts, among them J1 Conn_01x07, J3 Conn_01x05, SW1 RotaryEncoder_Switch, SW2 RotaryEncoder_Switch, U1 XC6206PxxxMR, U2 SRV05-4, U3 RP2040, U4 W25Q128JVS, Y1 Crystal_GND24

Commit message: commit chimera and associated plate directory
Other:
- board text added: "JLCJLCJLCJLC"
- board text added: "q9 chimera - xomm x baconspoon"
- board text added: "χίμαιρα"
