File: Q9-Chimera/Q9-Chimera-PCB/Q9-Chimera.kicad_sch (KiCad schematic)
At the start: 209 parts, among them J1 Conn_01x07, J2 USB_C_Receptacle_USB2.0_16P, J3 Conn_01x05, J4 Conn_01x04, SW1 RotaryEncoder_Switch, SW2 RotaryEncoder_Switch, U1 XC6206PxxxMR, U2 SRV05-4, U3 RP2040, U4 W25Q128JVS, Y1 Crystal_GND24

Commit message: testing more THT
Parts:
- MX52, MX66: footprint PCM_marbastlib-mx:SW_MX_HS_CPG151101S11_1u -> PCM_marbastlib-mx:SW_MX_1u
Changed lines of the file:
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@@
 			)
 		)
-		(property "Footprint" "PCM_marbastlib-mx:SW_MX_HS_CPG151101S11_1u"
+		(property "Footprint" "PCM_marbastlib-mx:SW_MX_1u"
 			(at 233.045 94.615 0)
 			(effects
@@
 			)
 		)
-		(property "Footprint" "PCM_marbastlib-mx:SW_MX_HS_CPG151101S11_1u"
+		(property "Footprint" "PCM_marbastlib-mx:SW_MX_1u"
 			(at 166.37 94.615 0)
 			(effects
