File: Q9-Chimera/Q9-Chimera-Plate/Q9-Chimera-Plate.kicad_pcb (KiCad board)
At the start: 2 copper layers, 312.5 x 90.5 mm, 0 parts

Commit message: split 225/275 to limousine, add 8u/10u support
Other:
- outline, holes or cut-outs redrawn
